File: blinkingLight/blinkingLight.kicad_pcb (KiCad board)
At the start: 2 copper layers, 50.8 x 50.8 mm, 11 parts, among them J1 Conn_02x03_Odd_Even, J2 Conn_01x02_Pin, Q1 BC548, U1 ICM7555xB

Commit message: push
Parts:
- C1: footprint Capacitor_THT:CP_Radial_D5.0mm_P2.50mm -> Capacitor_THT:CP_Radial_D8.0mm_P5.00mm
- R1: value 470 -> 1k; footprint Resistor_THT:R_Axial_DIN0204_L3.6mm_D1.6mm_P7.62mm_Horizontal -> Resistor_THT:R_Axial_DIN0309_L9.0mm_D3.2mm_P15.24mm_Horizontal
- R2: value 1k -> 4.7k; footprint Resistor_THT:R_Axial_DIN0204_L3.6mm_D1.6mm_P7.62mm_Horizontal -> Resistor_THT:R_Axial_DIN0309_L9.0mm_D3.2mm_P15.24mm_Horizontal
- R3, R4: footprint Resistor_THT:R_Axial_DIN0204_L3.6mm_D1.6mm_P7.62mm_Horizontal -> Resistor_THT:R_Axial_DIN0309_L9.0mm_D3.2mm_P15.24mm_Horizontal
- moved D1 25.4 mm to (138.4, 101.3)
- moved D2 25.4 mm to (113.0, 101.3)
- moved J1 2.54 mm to (124.5, 104.1)
- moved J2 2.54 mm to (142.9, 121.9)
- moved R1 2.54 mm to (111.8, 95.2)
- moved R2 2.54 mm to (119.4, 95.2)
- moved R3 2.54 mm to (127.0, 95.2)
- moved R4 2.54 mm to (144.8, 95.2)
- moved U1 2.54 mm to (121.9, 111.8)
- moved C1 2.54 mm to (110.5, 119.4)
- moved Q1 1.27 mm to (134.6, 87.6)
Connections:
- D1 pad 1: GND -> Net-(D1-K)
- D2 pad 2: Net-(D1-A) -> Net-(D1-K)
Routing:
- net Net-(D1-A): track 37.9 -> 7.62 mm, vias 2 -> 0
- net Net-(D1-K): track 0.00 -> 22.9 mm, vias 0 -> 2
- net Net-(Q1-B): track 60.2 -> 65.6 mm
- net GND: track 21.6 -> 17.2 mm
- net +9V: track 42.3 -> 46.1 mm
- net Net-(Q1-E): track 9.20 -> 10.8 mm
- net Net-(J1-Pin_1): track 17.8 -> 16.4 mm

Commit message: push
Parts:
- C1: footprint Capacitor_THT:CP_Radial_D8.0mm_P5.00mm -> Capacitor_THT:CP_Radial_D5.0mm_P2.00mm
- D1, D2: footprint LED_THT:LED_D3.0mm_Horizontal_O6.35mm_Z10.0mm -> LED_THT:LED_D5.0mm
- J1: footprint Connector_PinHeader_1.00mm:PinHeader_2x03_P1.00mm_Vertical -> Connector_PinHeader_2.54mm:PinHeader_2x03_P2.54mm_Vertical
- J2: footprint Jumper:SolderJumper-2_P1.3mm_Open_Pad1.0x1.5mm -> TerminalBlock:TerminalBlock_Xinya_XY308-2.54-2P_1x02_P2.54mm_Horizontal
- R1, R2, R3, R4: footprint Resistor_THT:R_Axial_DIN0309_L9.0mm_D3.2mm_P15.24mm_Horizontal -> Resistor_THT:R_Axial_DIN0207_L6.3mm_D2.5mm_P10.16mm_Horizontal
- moved Q1 29.3 mm to (132.1, 116.8)
- moved J1 19.8 mm to (111.8, 119.4)
- moved R3 18.2 mm to (119.4, 111.8)
- moved R4 17.3 mm to (139.7, 111.8)
- moved R2 17.3 mm to (114.3, 111.8)
- moved R1 16.7 mm to (109.2, 111.8)
- moved C1 14.2 mm to (124.5, 116.8)
- moved U1 8.51 mm to (125.7, 104.2)
- moved D2 7.92 mm to (108.0, 95.2)
- moved D1 7.89 mm to (143.5, 95.2)
- moved J2 3.47 mm to (141.2, 118.9)
Connections:
- C1 pad 1: Net-(U1-THR) -> GND
- C1 pad 2: GND -> Net-(Q1-B)
- U1 pad 6: Net-(U1-THR) -> Net-(Q1-B)
Routing:
- net +9V: track 46.1 -> 0.00 mm
- net Net-(U1-THR): track 22.2 -> 0.00 mm
- net GND: track 17.2 -> 0.00 mm, vias 1 -> 0
- net Net-(Q1-B): track 65.6 -> 50.0 mm, vias 2 -> 0
- net Net-(D1-A): track 7.62 -> 19.1 mm
- net Net-(D1-K): track 22.9 -> 33.0 mm, vias 2 -> 0
- net Net-(J1-Pin_3): track 17.1 -> 8.49 mm, vias 2 -> 0
- net Net-(J1-Pin_1): track 16.4 -> 8.67 mm
- net Net-(Q1-E): track 10.8 -> 17.3 mm
- net Net-(J1-Pin_2): track 20.2 -> 17.1 mm
Other:
- board text added: "UCF GLAMPING 2025"

Commit message: fixed
Parts:
- U1: footprint Package_DIP:DIP-6_W7.62mm -> Package_DIP:DIP-8_W7.62mm
- moved U1 2.86 mm to (124.5, 101.6)
- moved J2 0.85 mm to (141.6, 118.1)
Connections:
- C1 pad 1: GND -> Net-(Q1-B)
- C1 pad 2: Net-(Q1-B) -> GND
Routing:
- net +9V: track 0.00 -> 37.8 mm
- net Net-(Q1-B): track 50.0 -> 45.6 mm
- net Net-(J1-Pin_2): track 17.1 -> 18.4 mm
Other:
- board size 50.8 x 50.8 mm -> 44.4 x 40.6 mm
- board text added: "+"
