File: blinkingLight/blinkingLight.kicad_sch (KiCad schematic)
At the start: 11 parts, among them J1 Conn_02x03_Odd_Even, J2 Conn_01x02_Pin, Q1 BC548, U1 ICM7555xB

Commit message: push
Connections:
- net GND: no longer D1.1 (K)
- net at D1.2 (A), R4.1: no longer D2.2 (A)
- new net: D1.1 (K), D2.2 (A)
Other:
- moved on the sheet: C1, D1, D2
Changed lines of the file:
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@@
 	)
 	(junction
-		(at 96.52 111.76)
-		(diameter 0)
-		(color 0 0 0 0)
-	)
-	(junction
-		(at 104.14 111.76)
+		(at 120.65 111.76)
 		(diameter 0)
 		(color 0 0 0 0)
@@
 	)
 	(junction
-		(at 113.03 111.76)
-		(diameter 0)
-		(color 0 0 0 0)
-	)
-	(junction
 		(at 157.48 102.87)
 		(diameter 0)
@@
 	(wire
 		(pts
-			(xy 104.14 111.76) (xy 104.14 118.11)
-		)
-		(stroke
-			(width 0)
-			(type default)
-		)
-	)
-	(wire
-		(pts
 			(xy 80.01 111.76) (xy 69.85 111.76)
 		)
@@
 	(wire
 		(pts
-			(xy 104.14 111.76) (xy 113.03 111.76)
-		)
-		(stroke
-			(width 0)
-			(type default)
-		)
-	)
-	(wire
-		(pts
 			(xy 77.47 99.06) (xy 85.09 99.06)
 		)
@@
 	(wire
 		(pts
+			(xy 87.63 111.76) (xy 93.98 111.76)
+		)
+		(stroke
+			(width 0)
+			(type default)
+		)
+	)
+	(wire
+		(pts
 			(xy 134.62 102.87) (xy 134.62 93.98)
 		)
@@
 	(wire
 		(pts
-			(xy 96.52 106.68) (xy 96.52 111.76)
+			(xy 115.57 111.76) (xy 120.65 111.76)
 		)
 		(stroke
@@
 	(wire
 		(pts
-			(xy 120.65 111.76) (xy 170.18 111.76)
+			(xy 128.27 111.76) (xy 170.18 111.76)
 		)
 		(stroke
@@
 	(wire
 		(pts
-			(xy 96.52 111.76) (xy 96.52 118.11)
-		)
-		(stroke
-			(width 0)
-			(type default)
-		)
-	)
-	(wire
-		(pts
 			(xy 172.72 69.85) (xy 172.72 83.82)
 		)
@@
 	(wire
 		(pts
-			(xy 113.03 111.76) (xy 113.03 115.57)
+			(xy 120.65 111.76) (xy 120.65 115.57)
+		)
+		(stroke
+			(width 0)
+			(type default)
+		)
+	)
+	(wire
+		(pts
+			(xy 101.6 111.76) (xy 107.95 111.76)
 		)
 		(stroke
@@
 	(wire
 		(pts
-			(xy 96.52 111.76) (xy 87.63 111.76)
-		)
-		(stroke
-			(width 0)
-			(type default)
-		)
-	)
-	(wire
-		(pts
 			(xy 90.17 67.31) (xy 85.09 67.31)
 		)
@@
 		(pts
 			(xy 69.85 111.76) (xy 69.85 104.14)
-		)
-		(stroke
-			(width 0)
-			(type default)
-		)
-	)
-	(wire
-		(pts
-			(xy 104.14 106.68) (xy 104.14 111.76)
 		)
 		(stroke
@@
 	(symbol
 		(lib_id "Device:C")
-		(at 116.84 111.76 270)
+		(at 124.46 111.76 270)
 		(unit 1)
 		(exclude_from_sim no)
@@
 		(fields_autoplaced yes)
 		(property "Reference" "C1"
-			(at 116.84 104.14 90)
+			(at 124.46 104.14 90)
 			(effects
 				(font
@@
 		)
 		(property "Value" "100μF"
-			(at 116.84 106.68 90)
+			(at 124.46 106.68 90)
 			(effects
 				(font
@@
 		)
 		(property "Footprint" "Capacitor_THT:CP_Radial_D8.0mm_P5.00mm"
-			(at 113.03 112.7252 0)
+			(at 120.65 112.7252 0)
 			(effects
 				(font
@@
 		)
 		(property "Datasheet" "~"
-			(at 116.84 111.76 0)
+			(at 124.46 111.76 0)
 			(effects
 				(font
@@
 		)
 		(property "Description" "Unpolarized capacitor"
-			(at 116.84 111.76 0)
+			(at 124.46 111.76 0)
 			(effects
 				(font
@@
 	(symbol
 		(lib_id "Device:D")
-		(at 100.33 118.11 180)
+		(at 111.76 111.76 180)
 		(unit 1)
 		(exclude_from_sim no)
@@
 		(fields_autoplaced yes)
 		(property "Reference" "D2"
-			(at 100.33 111.76 0)
+			(at 111.76 105.41 0)
 			(effects
 				(font
@@
 		)
 		(property "Value" "D"
-			(at 100.33 114.3 0)
+			(at 111.76 107.95 0)
 			(effects
 				(font
@@
 		)
 		(property "Footprint" "LED_THT:LED_D3.0mm_Horizontal_O6.35mm_Z10.0mm"
-			(at 100.33 118.11 0)
+			(at 111.76 111.76 0)
 			(effects
 				(font
@@
 		)
 		(property "Datasheet" "~"
-			(at 100.33 118.11 0)
+			(at 111.76 111.76 0)
 			(effects
 				(font
@@
 		)
 		(property "Description" "Diode"
-			(at 100.33 118.11 0)
+			(at 111.76 111.76 0)
 			(effects
 				(font
@@
 		)
 		(property "Sim.Device" "D"
-			(at 100.33 118.11 0)
+			(at 111.76 111.76 0)
 			(effects
 				(font
@@
 		)
 		(property "Sim.Pins" "1=K 2=A"
-			(at 100.33 118.11 0)
+			(at 111.76 111.76 0)
 			(effects
 				(font
@@
 	(symbol
 		(lib_id "power:GND")
-		(at 113.03 115.57 0)
+		(at 120.65 115.57 0)
 		(unit 1)
 		(exclude_from_sim no)
@@
 		(fields_autoplaced yes)
 		(property "Reference" "#PWR03"
-			(at 113.03 121.92 0)
+			(at 120.65 121.92 0)
 			(effects
 				(font
@@
 		)
 		(property "Value" "GND"
-			(at 113.03 120.65 0)
+			(at 120.65 120.65 0)
 			(effects
 				(font
@@
 		)
 		(property "Footprint" ""
-			(at 113.03 115.57 0)
+			(at 120.65 115.57 0)
 			(effects
 				(font
@@
 		)
 		(property "Datasheet" ""
-			(at 113.03 115.57 0)
+			(at 120.65 115.57 0)
 			(effects
 				(font
@@
 		)
 		(property "Description" "Power symbol creates a global label with name \"GND\" , ground"
-			(at 113.03 115.57 0)
+			(at 120.65 115.57 0)
 			(effects
 				(font
@@
 	(symbol
 		(lib_id "Device:D")
-		(at 100.33 106.68 180)
+		(at 97.79 111.76 180)
 		(unit 1)
 		(exclude_from_sim no)
@@
 		(fields_autoplaced yes)
 		(property "Reference" "D1"
-			(at 100.33 100.33 0)
+			(at 97.79 105.41 0)
 			(effects
 				(font
@@
 		)
 		(property "Value" "D"
-			(at 100.33 102.87 0)
+			(at 97.79 107.95 0)
 			(effects
 				(font
@@
 		)
 		(property "Footprint" "LED_THT:LED_D3.0mm_Horizontal_O6.35mm_Z10.0mm"
-			(at 100.33 106.68 0)
+			(at 97.79 111.76 0)
 			(effects
 				(font
@@
 		)
 		(property "Datasheet" "~"
-			(at 100.33 106.68 0)
+			(at 97.79 111.76 0)
 			(effects
 				(font
@@
 		)
 		(property "Description" "Diode"
-			(at 100.33 106.68 0)
+			(at 97.79 111.76 0)
 			(effects
 				(font
@@
 		)
 		(property "Sim.Device" "D"
-			(at 100.33 106.68 0)
+			(at 97.79 111.76 0)
 			(effects
 				(font
@@
 		)
 		(property "Sim.Pins" "1=K 2=A"
-			(at 100.33 106.68 0)
-			(effects
-				(font
+			(at 97.79 111.76 0)
+			(effects
+				(font

Commit message: push
Parts:
- C1: symbol Device:C -> Device:C_Polarized
- R4: value 220 -> 100
Connections:
- net at Q1.2 (B), R1.2, R2.2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: now also C1.1, U1.6 (THR)
Other:
- note added: "0.85 seconds per blink"
- note added: "8.5 seconds per blink"
- moved on the sheet: D1, D2, J1, J2, R1, R2, R3, R4

Commit message: fixed
Parts:
- C1: footprint Capacitor_THT:CP_Radial_D8.0mm_P5.00mm -> Capacitor_THT:CP_Radial_D5.0mm_P2.00mm
- D1, D2: footprint LED_THT:LED_D3.0mm_Horizontal_O6.35mm_Z10.0mm -> LED_THT:LED_D5.0mm
- J1: footprint Connector_PinHeader_1.00mm:PinHeader_2x03_P1.00mm_Vertical -> Connector_PinHeader_2.54mm:PinHeader_2x03_P2.54mm_Vertical
- J2: footprint Jumper:SolderJumper-2_P1.3mm_Open_Pad1.0x1.5mm -> TerminalBlock:TerminalBlock_Xinya_XY308-2.54-2P_1x02_P2.54mm_Horizontal
- R1, R2, R3: footprint Resistor_THT:R_Axial_DIN0309_L9.0mm_D3.2mm_P15.24mm_Horizontal -> Resistor_THT:R_Axial_DIN0207_L6.3mm_D2.5mm_P10.16mm_Horizontal
- R4: value 100 -> 220; footprint Resistor_THT:R_Axial_DIN0309_L9.0mm_D3.2mm_P15.24mm_Horizontal -> Resistor_THT:R_Axial_DIN0207_L6.3mm_D2.5mm_P10.16mm_Horizontal
- U1: footprint Package_DIP:DIP-6_W7.62mm -> Package_DIP:DIP-8_W7.62mm
Changed lines of the file:
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@@
+	)
+	(junction
+		(at 157.48 102.87)
+		(diameter 0)
+		(color 0 0 0 0)
 	)
 	(junction
@@
 	(wire
 		(pts
+			(xy 163.83 49.53) (xy 157.48 49.53)
+		)
+		(stroke
+			(width 0)
+			(type default)
+		)
+	)
+	(wire
+		(pts
 			(xy 118.11 67.31) (xy 119.38 67.31)
 		)
@@
 		(pts
 			(xy 100.33 69.85) (xy 100.33 77.47)
+		)
+		(stroke
+			(width 0)
+			(type default)
+		)
+	)
+	(wire
+		(pts
+			(xy 157.48 102.87) (xy 165.1 102.87)
 		)
 		(stroke
@@
 			)
 		)
-		(property "Footprint" "Resistor_THT:R_Axial_DIN0309_L9.0mm_D3.2mm_P15.24mm_Horizontal"
+		(property "Footprint" "Resistor_THT:R_Axial_DIN0207_L6.3mm_D2.5mm_P10.16mm_Horizontal"
 			(at 96.52 87.122 90)
 			(effects
@@
 			)
 		)
-		(property "Footprint" "Jumper:SolderJumper-2_P1.3mm_Open_Pad1.0x1.5mm"
+		(property "Footprint" "TerminalBlock:TerminalBlock_Xinya_XY308-2.54-2P_1x02_P2.54mm_Horizontal"
 			(at 29.21 48.26 0)
 			(effects
@@
 			)
 		)
-		(property "Footprint" "Capacitor_THT:CP_Radial_D8.0mm_P5.00mm"
+		(property "Footprint" "Capacitor_THT:CP_Radial_D5.0mm_P2.00mm"
 			(at 91.7448 106.68 0)
 			(effects
@@
 			)
 		)
-		(property "Description" "Polarized capacitor"
+		(property "Description" "Unpolarized capacitor"
 			(at 92.71 102.87 0)
 			(effects
@@
 			)
 		)
-		(property "Footprint" "LED_THT:LED_D3.0mm_Horizontal_O6.35mm_Z10.0mm"
+		(property "Footprint" "LED_THT:LED_D5.0mm"
 			(at 69.85 130.81 0)
 			(effects
@@
 			)
 		)
-		(property "Footprint" "Resistor_THT:R_Axial_DIN0309_L9.0mm_D3.2mm_P15.24mm_Horizontal"
+		(property "Footprint" "Resistor_THT:R_Axial_DIN0207_L6.3mm_D2.5mm_P10.16mm_Horizontal"
 			(at 96.52 65.532 90)
 			(effects
@@
 			)
 		)
-		(property "Footprint" "LED_THT:LED_D3.0mm_Horizontal_O6.35mm_Z10.0mm"
+		(property "Footprint" "LED_THT:LED_D5.0mm"
 			(at 69.85 123.19 0)
 			(effects
@@
 			)
 		)
-		(property "Footprint" "Resistor_THT:R_Axial_DIN0309_L9.0mm_D3.2mm_P15.24mm_Horizontal"
+		(property "Footprint" "Resistor_THT:R_Axial_DIN0207_L6.3mm_D2.5mm_P10.16mm_Horizontal"
 			(at 96.52 75.692 90)
 			(effects
@@
 			)
 		)
-		(property "Footprint" "Connector_PinHeader_1.00mm:PinHeader_2x03_P1.00mm_Vertical"
+		(property "Footprint" "Connector_PinHeader_2.54mm:PinHeader_2x03_P2.54mm_Vertical"
 			(at 110.49 69.85 0)
 			(effects
@@
 			)
 		)
-		(property "Value" "100"
+		(property "Value" "220"
 			(at 72.39 116.8399 0)
 			(effects
@@
 			)
 		)
-		(property "Footprint" "Resistor_THT:R_Axial_DIN0309_L9.0mm_D3.2mm_P15.24mm_Horizontal"
+		(property "Footprint" "Resistor_THT:R_Axial_DIN0207_L6.3mm_D2.5mm_P10.16mm_Horizontal"
 			(at 71.628 115.57 90)
 			(effects
@@
 	)
 	(symbol
+		(lib_id "power:PWR_FLAG")
+		(at 165.1 102.87 0)
+		(unit 1)
+		(exclude_from_sim no)
+		(in_bom yes)
+		(on_board yes)
+		(dnp no)
+		(fields_autoplaced yes)
+		(property "Reference" "#FLG02"
+			(at 165.1 100.965 0)
+			(effects
+				(font
+					(size 1.27 1.27)
+				)
+				(hide yes)
+			)
+		)
+		(property "Value" "PWR_FLAG"
+			(at 165.1 97.79 0)
+			(effects
+				(font
+					(size 1.27 1.27)
+				)
+			)
+		)
+		(property "Footprint" ""
+			(at 165.1 102.87 0)
+			(effects
+				(font
+					(size 1.27 1.27)
+				)
+				(hide yes)
+			)
+		)
+		(property "Datasheet" "~"
+			(at 165.1 102.87 0)
+			(effects
+				(font
+					(size 1.27 1.27)
+				)
+				(hide yes)
+			)
+		)
+		(property "Description" "Special symbol for telling ERC where power comes from"
+			(at 165.1 102.87 0)
+			(effects
+				(font
+					(size 1.27 1.27)
+				)
+				(hide yes)
+			)
+		)
+		(pin "1"
+		)
+		(instances
+			(project ""
+				(path "/c44aec96-1bce-4271-9432-231eb29dd86b"
+					(reference "#FLG02")
+					(unit 1)
+				)
+			)
+		)
+	)
+	(symbol
 		(lib_id "Timer:ICM7555xB")
 		(at 157.48 88.9 0)
@@
 			)
 		)
-		(property "Footprint" "Package_DIP:DIP-6_W7.62mm"
+		(property "Footprint" "Package_DIP:DIP-8_W7.62mm"
 			(at 179.07 99.06 0)
 			(effects
@@
 					(unit 1)
 				)
+			)
+		)
+	)
+	(symbol
+		(lib_id "power:PWR_FLAG")
+		(at 163.83 49.53 0)
+		(unit 1)
+		(exclude_from_sim no)
+		(in_bom yes)
+		(on_board yes)
+		(dnp no)
+		(fields_autoplaced yes)
+		(property "Reference" "#FLG01"
+			(at 163.83 47.625 0)
+			(effects
+				(font
+					(size 1.27 1.27)
+				)
+				(hide yes)
+			)
+		)
+		(property "Value" "PWR_FLAG"
+			(at 163.83 44.45 0)
+			(effects
+				(font
+					(size 1.27 1.27)
+				)
+			)
+		)
+		(property "Footprint" ""
+			(at 163.83 49.53 0)
+			(effects
+				(font
+					(size 1.27 1.27)
+				)
+				(hide yes)
+			)
+		)
+		(property "Datasheet" "~"
+			(at 163.83 49.53 0)
+			(effects
+				(font
+					(size 1.27 1.27)
+				)
+				(hide yes)
+			)
+		)
+		(property "Description" "Special symbol for telling ERC where power comes from"
+			(at 163.83 49.53 0)
+			(effects
+				(font
+					(size 1.27 1.27)
+				)
+				(hide yes)
+			)
+		)
+		(pin "1"
+		)
+		(instances
+			(project ""
+				(path "/c44aec96-1bce-4271-9432-231eb29dd86b"
+					(reference "#FLG01")
+					(unit 1)
+				)

Commit message: updated value
Parts:
- R4: value 220 -> 100
Changed lines of the file:
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@@
 			)
 		)
-		(property "Value" "220"
+		(property "Value" "100"
 			(at 72.39 116.8399 0)
 			(effects
